File: motor_unicorn.kicad_sch (KiCad schematic)
At the start: 18 parts, among them J10 Conn_01x06_Pin, J5 Conn_01x03_Socket, J6 Conn_01x03_Socket, J7 Conn_01x06_Pin, J8 Conn_01x06_Pin, J9 Conn_01x06_Pin, U16 OLED

Commit message: ordered version
Parts:
- C42: footprint Capacitor_SMD:C_0402_1005Metric -> Capacitor_SMD:C_0805_2012Metric
- R26, R27: LCSC (none) -> C25744
Changed lines of the file:
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@@
+			)
+		)
+		(property "LCSC" "C25744"
+			(at 223.52 54.6099 0)
+			(effects
+				(font
+					(size 1.27 1.27)
+				)
+				(hide yes)
 			)
 		)
@@
 			)
 		)
+		(property "LCSC" "C25744"
+			(at 240.03 54.6099 0)
+			(effects
+				(font
+					(size 1.27 1.27)
+				)
+				(hide yes)
+			)
+		)
 		(pin "1"
 		)
@@
 			)
 		)
-		(property "Footprint" "Capacitor_SMD:C_0402_1005Metric"
+		(property "Footprint" "Capacitor_SMD:C_0805_2012Metric"
 			(at 25.0952 182.88 0)
 			(effects

Commit message: tiny last minute fixes
Parts:
- R26, R27: LCSC C25744 -> (none)
Changed lines of the file:
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@@
-			)
-		)
-		(property "LCSC" "C25744"
-			(at 223.52 54.6099 0)
-			(effects
-				(font
-					(size 1.27 1.27)
-				)
-				(hide yes)
 			)
 		)
@@
 			(effects
 				(font
-					(size 1.27 1.27)
-				)
-				(hide yes)
-			)
-		)
-		(property "LCSC" "C25744"
-			(at 240.03 54.6099 0)
-			(effects
-				(font
