File: bridge.kicad_sch (KiCad schematic)
At the start: 14 parts

Commit message: finalized the design
Parts:
- removed TP11, TP5, TP6, TP7: TestPoint, symbol Connector:TestPoint
- removed U21, U24: ~, Package_DFN_QFN:PQFN-8-EP_6x5mm_P1.27mm_Generic, symbol unicorn_lib:CJAC150N03A
- added C52: 100u, Capacitor_SMD:CP_Elec_6.3x7.7, symbol Device:C_Polarized
- added Q5, Q8: Q_NMOS_SGD, unicorn_footprints:PQFN-8-EP_6x5mm_P1.27mm_Generic, symbol Device:Q_NMOS_SGD
- C23: value 100nF -> 100n; footprint (none) -> Capacitor_SMD:C_0402_1005Metric
- C24: value 10uF -> 10u; footprint (none) -> Capacitor_SMD:C_0603_1608Metric
- D4, D5, D7: footprint (none) -> Diode_SMD:D_SOD-323
- R10, R9: footprint (none) -> Resistor_SMD:R_0402_1005Metric
- U5: value ~ -> EG2132; footprint (none) -> Package_SO:SSOP-8_3.9x5.05mm_P1.27mm
Connections:
- net GND: now also C52.2, Q5.1 (S)
- net OUT: now also Q5.3 (D), Q8.1 (S)
- net VPP: now also C52.1, Q8.3 (D)
- net at D7.2 (A), R10.2: now also Q8.2 (G)
- net at D4.2 (A), R9.2: now also Q5.2 (G)
