File: cur_sense.kicad_sch (KiCad schematic)
At the start: 3 parts, among them U7 INA240A3D

Commit message: finalized the design
Parts:
- R14: value R -> 5mR; footprint (none) -> Resistor_SMD:R_2512_6332Metric; LSCS (none) -> C309526
- U7: value INA240A3D -> INA240A1D
Changed lines of the file:
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@@
-					(unit 1)
-				)
-				(path "/0a1df5c3-2d18-40b4-a193-f71ff4161835/f60af36c-b1a2-42b2-91f5-eecb1fb4b462"
-					(reference "#PWR081")
 					(unit 1)
 				)
@@
 				)
 				(path "/0a1df5c3-2d18-40b4-a193-f71ff4161835/a7414898-e1cd-499f-ba5d-c57d53dd7e89"
+					(reference "#PWR0171")
+					(unit 1)
+				)
+				(path "/0a1df5c3-2d18-40b4-a193-f71ff4161835/f60af36c-b1a2-42b2-91f5-eecb1fb4b462"
 					(reference "#PWR0128")
 					(unit 1)
@@
 					(unit 1)
 				)
-				(path "/0a1df5c3-2d18-40b4-a193-f71ff4161835/f60af36c-b1a2-42b2-91f5-eecb1fb4b462"
-					(reference "#PWR080")
-					(unit 1)
-				)
 				(path "/0a1df5c3-2d18-40b4-a193-f71ff4161835/7c01ea32-a0ec-4edf-98d7-077b83babfaf"
 					(reference "#PWR0122")
@@
 				)
 				(path "/0a1df5c3-2d18-40b4-a193-f71ff4161835/a7414898-e1cd-499f-ba5d-c57d53dd7e89"
+					(reference "#PWR0175")
+					(unit 1)
+				)
+				(path "/0a1df5c3-2d18-40b4-a193-f71ff4161835/f60af36c-b1a2-42b2-91f5-eecb1fb4b462"
 					(reference "#PWR0127")
 					(unit 1)
@@
 					(unit 1)
 				)
-				(path "/0a1df5c3-2d18-40b4-a193-f71ff4161835/f60af36c-b1a2-42b2-91f5-eecb1fb4b462"
-					(reference "#PWR079")
-					(unit 1)
-				)
 				(path "/0a1df5c3-2d18-40b4-a193-f71ff4161835/7c01ea32-a0ec-4edf-98d7-077b83babfaf"
 					(reference "#PWR0121")
@@
 				)
 				(path "/0a1df5c3-2d18-40b4-a193-f71ff4161835/a7414898-e1cd-499f-ba5d-c57d53dd7e89"
+					(reference "#PWR0174")
+					(unit 1)
+				)
+				(path "/0a1df5c3-2d18-40b4-a193-f71ff4161835/f60af36c-b1a2-42b2-91f5-eecb1fb4b462"
 					(reference "#PWR0126")
 					(unit 1)
@@
 					(unit 1)
 				)
-				(path "/0a1df5c3-2d18-40b4-a193-f71ff4161835/f60af36c-b1a2-42b2-91f5-eecb1fb4b462"
-					(reference "#PWR078")
-					(unit 1)
-				)
 				(path "/0a1df5c3-2d18-40b4-a193-f71ff4161835/7c01ea32-a0ec-4edf-98d7-077b83babfaf"
 					(reference "#PWR0120")
@@
 				)
 				(path "/0a1df5c3-2d18-40b4-a193-f71ff4161835/a7414898-e1cd-499f-ba5d-c57d53dd7e89"
+					(reference "#PWR0173")
+					(unit 1)
+				)
+				(path "/0a1df5c3-2d18-40b4-a193-f71ff4161835/f60af36c-b1a2-42b2-91f5-eecb1fb4b462"
 					(reference "#PWR0125")
 					(unit 1)
@@
 					(unit 1)
 				)
+				(path "/0a1df5c3-2d18-40b4-a193-f71ff4161835/7c01ea32-a0ec-4edf-98d7-077b83babfaf"
+					(reference "C38")
+					(unit 1)
+				)
+				(path "/0a1df5c3-2d18-40b4-a193-f71ff4161835/a7414898-e1cd-499f-ba5d-c57d53dd7e89"
+					(reference "C39")
+					(unit 1)
+				)
 				(path "/0a1df5c3-2d18-40b4-a193-f71ff4161835/f60af36c-b1a2-42b2-91f5-eecb1fb4b462"
 					(reference "C28")
-					(unit 1)
-				)
-				(path "/0a1df5c3-2d18-40b4-a193-f71ff4161835/7c01ea32-a0ec-4edf-98d7-077b83babfaf"
-					(reference "C38")
-					(unit 1)
-				)
-				(path "/0a1df5c3-2d18-40b4-a193-f71ff4161835/a7414898-e1cd-499f-ba5d-c57d53dd7e89"
-					(reference "C39")
 					(unit 1)
 				)
@@
 			)
 		)
-		(property "Value" "INA240A3D"
+		(property "Value" "INA240A1D"
 			(at 65.278 40.894 0)
 			(effects
@@
 					(unit 1)
 				)
+				(path "/0a1df5c3-2d18-40b4-a193-f71ff4161835/7c01ea32-a0ec-4edf-98d7-077b83babfaf"
+					(reference "U14")
+					(unit 1)
+				)
+				(path "/0a1df5c3-2d18-40b4-a193-f71ff4161835/a7414898-e1cd-499f-ba5d-c57d53dd7e89"
+					(reference "U15")
+					(unit 1)
+				)
 				(path "/0a1df5c3-2d18-40b4-a193-f71ff4161835/f60af36c-b1a2-42b2-91f5-eecb1fb4b462"
 					(reference "U8")
-					(unit 1)
-				)
-				(path "/0a1df5c3-2d18-40b4-a193-f71ff4161835/7c01ea32-a0ec-4edf-98d7-077b83babfaf"
-					(reference "U14")
-					(unit 1)
-				)
-				(path "/0a1df5c3-2d18-40b4-a193-f71ff4161835/a7414898-e1cd-499f-ba5d-c57d53dd7e89"
-					(reference "U15")
 					(unit 1)
 				)
@@
 					(unit 1)
 				)
-				(path "/0a1df5c3-2d18-40b4-a193-f71ff4161835/f60af36c-b1a2-42b2-91f5-eecb1fb4b462"
-					(reference "#PWR082")
-					(unit 1)
-				)
 				(path "/0a1df5c3-2d18-40b4-a193-f71ff4161835/7c01ea32-a0ec-4edf-98d7-077b83babfaf"
 					(reference "#PWR0124")
@@
 				)
 				(path "/0a1df5c3-2d18-40b4-a193-f71ff4161835/a7414898-e1cd-499f-ba5d-c57d53dd7e89"
+					(reference "#PWR0172")
+					(unit 1)
+				)
+				(path "/0a1df5c3-2d18-40b4-a193-f71ff4161835/f60af36c-b1a2-42b2-91f5-eecb1fb4b462"
 					(reference "#PWR0129")
 					(unit 1)
@@
 			)
 		)
-		(property "Value" "R"
+		(property "Value" "5mR"
 			(at 43.18 48.2599 0)
 			(effects
@@
 			)
 		)
-		(property "Footprint" ""
+		(property "Footprint" "Resistor_SMD:R_2512_6332Metric"
 			(at 38.862 46.99 90)
 			(effects
@@
 			)
 		)
+		(property "LSCS" "C309526"
+			(at 40.64 46.99 0)
+			(effects
+				(font
+					(size 1.27 1.27)
+				)
+				(hide yes)
+			)
+		)
+		(property "Feld6" ""
+			(at 40.64 46.99 0)
+			(effects
+				(font
+					(size 1.27 1.27)
+				)
+				(hide yes)
+			)
+		)
 		(pin "2"
 		)
@@
 					(unit 1)
 				)
+				(path "/0a1df5c3-2d18-40b4-a193-f71ff4161835/7c01ea32-a0ec-4edf-98d7-077b83babfaf"
+					(reference "R24")
+					(unit 1)
+				)
+				(path "/0a1df5c3-2d18-40b4-a193-f71ff4161835/a7414898-e1cd-499f-ba5d-c57d53dd7e89"
+					(reference "R25")
+					(unit 1)
+				)
 				(path "/0a1df5c3-2d18-40b4-a193-f71ff4161835/f60af36c-b1a2-42b2-91f5-eecb1fb4b462"
 					(reference "R15")
 					(unit 1)
 				)
-				(path "/0a1df5c3-2d18-40b4-a193-f71ff4161835/7c01ea32-a0ec-4edf-98d7-077b83babfaf"
-					(reference "R24")
-					(unit 1)
-				)
-				(path "/0a1df5c3-2d18-40b4-a193-f71ff4161835/a7414898-e1cd-499f-ba5d-c57d53dd7e89"
-					(reference "R25")
-					(unit 1)
-				)
