File: imu.kicad_sch (KiCad schematic)
At the start: 3 parts, among them U10 QMI8658

Commit message: finalized the design
Parts:
- U10: symbol vib_sense:QMI8658 -> unicorn_lib:QMI8658
Connections:
- net GND: now also U10.6 (GND), U10.7 (GND); no longer U10.6,7 (GND)
Changed lines of the file:
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@@
+	(wire
+		(pts
+			(xy 58.42 52.07) (xy 58.42 54.61)
+		)
+		(stroke
+			(width 0)
+			(type default)
+		)
+	)
 	(wire
 		(pts
@@
 	)
 	(symbol
-		(lib_id "vib_sense:QMI8658")
+		(lib_id "unicorn_lib:QMI8658")
 		(at 53.34 41.91 0)
 		(unit 1)
@@
 		(fields_autoplaced yes)
 		(property "Reference" "U10"
-			(at 58.0741 32.6969 0)
+			(at 58.0741 29.21 0)
 			(effects
 				(font
@@
 		)
 		(property "Value" "QMI8658"
-			(at 53.34 43.18 0)
-			(effects
-				(font
-					(size 1.27 1.27)
-				)
+			(at 58.0741 31.75 0)
+			(effects
+				(font
+					(size 1.27 1.27)
+				)
+				(justify left)
 			)
 		)
@@
 		(pin "5"
 		)
-		(pin "6,7"
+		(pin "6"
 		)
 		(pin "8"
 		)
 		(pin "9"
+		)
+		(pin "7"
 		)
 		(instances
@@
 					(unit 1)
 				)
+			)
+		)
+	)
+	(symbol
+		(lib_id "power:GND")
+		(at 58.42 54.61 0)
+		(unit 1)
+		(exclude_from_sim no)
+		(in_bom yes)
+		(on_board yes)
+		(dnp no)
+		(fields_autoplaced yes)
+		(property "Reference" "#PWR011"
+			(at 58.42 60.96 0)
+			(effects
+				(font
+					(size 1.27 1.27)
+				)
+				(hide yes)
+			)
+		)
+		(property "Value" "GND"
+			(at 58.42 58.7431 0)
+			(effects
+				(font
+					(size 1.27 1.27)
+				)
+			)
+		)
+		(property "Footprint" ""
+			(at 58.42 54.61 0)
+			(effects
+				(font
+					(size 1.27 1.27)
+				)
+				(hide yes)
+			)
+		)
+		(property "Datasheet" ""
+			(at 58.42 54.61 0)
+			(effects
+				(font
+					(size 1.27 1.27)
+				)
+				(hide yes)
+			)
+		)
+		(property "Description" ""
+			(at 58.42 54.61 0)
+			(effects
+				(font
+					(size 1.27 1.27)
+				)
+				(hide yes)
+			)
+		)
+		(pin "1"
+		)
+		(instances
+			(project "motor_unicorn"
+				(path "/0a1df5c3-2d18-40b4-a193-f71ff4161835/ca7056ea-07de-4c61-9685-e1c0e4cd1c9a"
+					(reference "#PWR011")
+					(unit 1)
+				)
