File: rp2040.kicad_sch (KiCad schematic)
At the start: 41 parts, among them J1 CON_SWD, J2 USB_C_Receptacle_USB2.0, SW1 SW_Push, U1 TLV62568DRL, U2 W25Q16JVUXIQ, U3 RP2040, Y1 12MHz

Commit message: more connections
Connections:
- net HALL_CSN: now reaches U3.27 (GPIO16)
- net HALL_CLK: now reaches U3.28 (GPIO17)
- net HALL_DAT_0: now reaches U3.29 (GPIO18)
- net HALL_DAT_1: now reaches U3.30 (GPIO19)
- net HALL_DAT_2: now reaches U3.31 (GPIO20)
- net HALL_DAT_3: now reaches U3.32 (GPIO21)
- net DISP_RES: now reaches U3.36 (GPIO24)
- no-connect marks 3 -> 4
Changed lines of the file:
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@@
 	)
 	(junction
+		(at 69.85 143.51)
+		(diameter 0)
+		(color 0 0 0 0)
+	)
+	(junction
 		(at 34.29 83.82)
 		(diameter 0)
@@
 	)
 	(no_connect
+		(at 207.01 45.72)
+	)
+	(no_connect
 		(at 113.03 50.8)
 	)
@@
 	(wire
 		(pts
+			(xy 69.85 137.16) (xy 69.85 143.51)
+		)
+		(stroke
+			(width 0)
+			(type default)
+		)
+	)
+	(wire
+		(pts
 			(xy 204.47 114.3) (xy 207.01 114.3)
 		)
@@
 	(wire
 		(pts
+			(xy 257.81 93.98) (xy 260.35 93.98)
+		)
+		(stroke
+			(width 0)
+			(type default)
+		)
+	)
+	(wire
+		(pts
 			(xy 237.49 35.56) (xy 237.49 38.1)
 		)
@@
 	(wire
 		(pts
+			(xy 257.81 91.44) (xy 260.35 91.44)
+		)
+		(stroke
+			(width 0)
+			(type default)
+		)
+	)
+	(wire
+		(pts
 			(xy 46.99 146.05) (xy 54.61 146.05)
 		)
@@
 	(wire
 		(pts
+			(xy 69.85 143.51) (xy 72.39 143.51)
+		)
+		(stroke
+			(width 0)
+			(type default)
+		)
+	)
+	(wire
+		(pts
 			(xy 147.32 54.61) (xy 147.32 55.88)
 		)
@@
 	(wire
 		(pts
+			(xy 257.81 106.68) (xy 260.35 106.68)
+		)
+		(stroke
+			(width 0)
+			(type default)
+		)
+	)
+	(wire
+		(pts
 			(xy 54.61 153.67) (xy 63.5 153.67)
 		)
@@
 	(wire
 		(pts
-			(xy 63.5 143.51) (xy 72.39 143.51)
+			(xy 63.5 143.51) (xy 69.85 143.51)
 		)
 		(stroke
@@
 		)
 	)
+	(wire
+		(pts
+			(xy 257.81 99.06) (xy 260.35 99.06)
+		)
+		(stroke
+			(width 0)
+			(type default)
+		)
+	)
+	(wire
+		(pts
+			(xy 257.81 96.52) (xy 260.35 96.52)
+		)
+		(stroke
+			(width 0)
+			(type default)
+		)
+	)
 	(polyline
 		(pts
@@
 	(wire
 		(pts
+			(xy 257.81 88.9) (xy 260.35 88.9)
+		)
+		(stroke
+			(width 0)
+			(type default)
+		)
+	)
+	(wire
+		(pts
 			(xy 115.57 43.18) (xy 115.57 40.64)
 		)
@@
 	(wire
 		(pts
+			(xy 257.81 86.36) (xy 260.35 86.36)
+		)
+		(stroke
+			(width 0)
+			(type default)
+		)
+	)
+	(wire
+		(pts
 			(xy 72.39 152.4) (xy 72.39 154.94)
 		)
@@
 		)
 	)
+	(hierarchical_label "HALL_DAT_2"
+		(shape input)
+		(at 260.35 96.52 0)
+		(fields_autoplaced yes)
+		(effects
+			(font
+				(size 1.27 1.27)
+			)
+			(justify left)
+		)
+	)
 	(hierarchical_label "PWM_L_1"
 		(shape output)
@@
 		)
 	)
+	(hierarchical_label "HALL_CLK"
+		(shape output)
+		(at 260.35 88.9 0)
+		(fields_autoplaced yes)
+		(effects
+			(font
+				(size 1.27 1.27)
+			)
+			(justify left)
+		)
+	)
 	(hierarchical_label "PWM_H_0"
 		(shape output)
@@
 		)
 	)
+	(hierarchical_label "HALL_DAT_3"
+		(shape input)
+		(at 260.35 99.06 0)
+		(fields_autoplaced yes)
+		(effects
+			(font
+				(size 1.27 1.27)
+			)
+			(justify left)
+		)
+	)
 	(hierarchical_label "PWM_L_5"
 		(shape output)
@@
 		)
 	)
+	(hierarchical_label "HALL_DAT_0"
+		(shape input)
+		(at 260.35 91.44 0)
+		(fields_autoplaced yes)
+		(effects
+			(font
+				(size 1.27 1.27)
+			)
+			(justify left)
+		)
+	)
 	(hierarchical_label "PWM_H_4"
 		(shape output)
@@
 		)
 	)
+	(hierarchical_label "DISP_RES"
+		(shape output)
+		(at 260.35 106.68 0)
+		(fields_autoplaced yes)
+		(effects
+			(font
+				(size 1.27 1.27)
+			)
+			(justify left)
+		)
+	)
+	(hierarchical_label "HALL_DAT_1"
+		(shape input)
+		(at 260.35 93.98 0)
+		(fields_autoplaced yes)
+		(effects
+			(font
+				(size 1.27 1.27)
+			)
+			(justify left)
+		)
+	)
 	(hierarchical_label "RS485_TX"
 		(shape output)
@@
 		)
 	)
+	(hierarchical_label "HALL_CSN"
+		(shape output)
+		(at 260.35 86.36 0)
+		(fields_autoplaced yes)
+		(effects
+			(font
+				(size 1.27 1.27)
+			)
+			(justify left)
+		)
+	)
 	(hierarchical_label "I2C_SDA"
 		(shape bidirectional)
@@
 					(unit 1)
 				)
+			)
+		)
+	)
+	(symbol
+		(lib_id "power:PWR_FLAG")
+		(at 69.85 137.16 0)
+		(unit 1)
+		(exclude_from_sim no)
+		(in_bom yes)
+		(on_board yes)
+		(dnp no)
+		(fields_autoplaced yes)
+		(property "Reference" "#FLG04"
+			(at 69.85 135.255 0)
+			(effects
+				(font
+					(size 1.27 1.27)
+				)
+				(hide yes)
+			)
+		)
+		(property "Value" "PWR_FLAG"
+			(at 69.85 132.08 0)
+			(effects
+				(font
+					(size 1.27 1.27)
+				)
+				(hide yes)
+			)
+		)
+		(property "Footprint" ""
+			(at 69.85 137.16 0)
+			(effects
+				(font
+					(size 1.27 1.27)
+				)
+				(hide yes)
+			)
+		)
+		(property "Datasheet" "~"
+			(at 69.85 137.16 0)
+			(effects
+				(font
+					(size 1.27 1.27)
+				)
+				(hide yes)
+			)
+		)
+		(property "Description" "Special symbol for telling ERC where power comes from"
+			(at 69.85 137.16 0)
+			(effects
+				(font
+					(size 1.27 1.27)
+				)
+				(hide yes)
+			)
+		)
+		(pin "1"
+		)
+		(instances
+			(project "motor_unicorn"
+				(path "/0a1df5c3-2d18-40b4-a193-f71ff4161835/82afce1c-e9f1-4e79-92a2-91123355c306"
+					(reference "#FLG04")
+					(unit 1)
+				)

Commit message: finalized the design
Parts:
- removed D2: D, Package_TO_SOT_SMD:SOT-723, symbol Device:D
- removed TP1, TP2, TP3: TestPoint, TestPoint:TestPoint_Pad_D1.0mm, symbol Connector:TestPoint
- added D2: D_Schottky, Diode_SMD:D_SOD-323, symbol Device:D_Schottky
- C1: footprint Capacitor_SMD:C_0603_1608Metric -> Capacitor_SMD:C_0402_1005Metric
- D1: footprint icon:XL-1010RGBC-WS2812B -> unicorn_footprints:XL-1010RGBC-WS2812B
- FB1: footprint Capacitor_SMD:C_0603_1608Metric -> Inductor_SMD:L_0603_1608Metric
- J1: LSCS (none) -> C2845371
- R3, SW1: now not fitted; now left out of the parts list
Connections:
- net +5V: now also D2.1 (K)
- net ADC_0: now also U3.41 (GPIO29_ADC3); no longer U3.38 (GPIO26_ADC0)
- net ADC_1: now also U3.40 (GPIO28_ADC2); no longer U3.39 (GPIO27_ADC1)
- net ADC_2: now also U3.39 (GPIO27_ADC1); no longer U3.40 (GPIO28_ADC2)
- net ADC_3: now also U3.38 (GPIO26_ADC0); no longer U3.41 (GPIO29_ADC3)
- net HALL_DAT_0: now also U3.31 (GPIO20); no longer U3.29 (GPIO18)
- net HALL_DAT_1: now also U3.32 (GPIO21); no longer U3.30 (GPIO19)
- net HALL_DAT_2: now also U3.29 (GPIO18); no longer U3.31 (GPIO20)
- net HALL_DAT_3: now also U3.30 (GPIO19); no longer U3.32 (GPIO21)
- net PWM_H_0: now also U3.14 (GPIO11); no longer U3.7 (GPIO5)
- net PWM_H_3: now also U3.2 (GPIO0); no longer U3.14 (GPIO11)
- net PWM_H_4: now also U3.6 (GPIO4); no longer U3.16 (GPIO13)
- net PWM_H_5: now also U3.4 (GPIO2); no longer U3.18 (GPIO15)
- net PWM_L_0: now also U3.13 (GPIO10); no longer U3.6 (GPIO4)
- net PWM_L_3: now also U3.3 (GPIO1); no longer U3.13 (GPIO10)
- net PWM_L_4: now also U3.7 (GPIO5); no longer U3.15 (GPIO12)
- net PWM_L_5: now also U3.5 (GPIO3); no longer U3.17 (GPIO14)
- net RS485_DE: now also U3.17 (GPIO14); no longer U3.4 (GPIO2)
- net RS485_NRE: now also U3.18 (GPIO15); no longer U3.5 (GPIO3)
- net RS485_RX: now also U3.16 (GPIO13); no longer U3.3 (GPIO1)
- net RS485_TX: now also U3.15 (GPIO12); no longer U3.2 (GPIO0)
- net at J2.A4 (VBUS), J2.A9 (VBUS), J2.B4 (VBUS)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: now also D2.2 (A)
- net USB_DIN_N: now reaches J2.A7 (D-), J2.B7 (D-), R4.1
- net USB_DIN_P: now reaches J2.A6 (D+), J2.B6 (D+), R5.1
- net USB_DM renamed USB_D-
- net USB_DP renamed USB_D+

Commit message: ordered version
Parts:
- J1: symbol Connector:Conn_01x03_Male -> Connector:Conn_01x03_Pin
- J2: symbol Connector:USB_C_Receptacle_USB2.0 -> Connector:USB_C_Receptacle_USB2.0_14P
- Y1: footprint Crystal:Crystal_SMD_TXC_7M-4Pin_3.2x2.5mm -> Crystal:Crystal_SMD_3225-4Pin_3.2x2.5mm
Connections:
- no-connect marks 4 -> 2
Other:
- moved on the sheet: U2
