File: rs485.kicad_sch (KiCad schematic)
At the start: 6 parts, among them J3 Conn_01x02_Socket, J4 Conn_01x02_Socket, U9 SIT3088E

Commit message: finalized the design
Parts:
- J3: footprint (none) -> Connector_Molex:Molex_PicoBlade_53398-0271_1x02-1MP_P1.25mm_Vertical; LCSC (none) -> C395343
- J4: footprint (none) -> Connector_Molex:Molex_PicoBlade_53398-0271_1x02-1MP_P1.25mm_Vertical
- R16: value 5k -> 1k
- U9: footprint icon:DFN8-3x3mm -> unicorn_footprints:DFN8-3x3mm
Connections:
- net at R16.1, U9.6 (A): now also J3.1 (Pin_1), J4.1 (Pin_1); no longer J3.2 (Pin_2), J4.2 (Pin_2)
- net at R17.2, U9.7 (B): now also J3.2 (Pin_2), J4.2 (Pin_2); no longer J3.1 (Pin_1), J4.1 (Pin_1)
Changed lines of the file:
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@@
 			)
 		)
-		(property "Value" "5k"
+		(property "Value" "1k"
 			(at 77.47 31.75 90)
 			(effects
@@
 			)
 		)
-		(property "Footprint" "icon:DFN8-3x3mm"
+		(property "Footprint" "unicorn_footprints:DFN8-3x3mm"
 			(at 60.96 59.69 0)
 			(effects
@@
 	(symbol
 		(lib_id "Connector:Conn_01x02_Socket")
-		(at 104.14 46.99 0)
-		(unit 1)
-		(exclude_from_sim no)
-		(in_bom yes)
-		(on_board yes)
-		(dnp no)
-		(fields_autoplaced yes)
+		(at 104.14 49.53 0)
+		(mirror x)
+		(unit 1)
+		(exclude_from_sim no)
+		(in_bom yes)
+		(on_board yes)
+		(dnp no)
 		(property "Reference" "J4"
-			(at 105.41 46.9899 0)
+			(at 105.41 49.5301 0)
 			(effects
 				(font
@@
 		)
 		(property "Value" "Conn_01x02_Socket"
-			(at 105.41 49.5299 0)
-			(effects
-				(font
-					(size 1.27 1.27)
-				)
-				(justify left)
-			)
-		)
-		(property "Footprint" ""
-			(at 104.14 46.99 0)
+			(at 105.41 46.9901 0)
+			(effects
+				(font
+					(size 1.27 1.27)
+				)
+				(justify left)
+			)
+		)
+		(property "Footprint" "Connector_Molex:Molex_PicoBlade_53398-0271_1x02-1MP_P1.25mm_Vertical"
+			(at 104.14 49.53 0)
 			(effects
 				(font
@@
 		)
 		(property "Datasheet" "~"
-			(at 104.14 46.99 0)
+			(at 104.14 49.53 0)
 			(effects
 				(font
@@
 		)
 		(property "Description" "Generic connector, single row, 01x02, script generated"
-			(at 104.14 46.99 0)
+			(at 104.14 49.53 0)
 			(effects
 				(font
@@
 	(symbol
 		(lib_id "Connector:Conn_01x02_Socket")
-		(at 104.14 39.37 0)
-		(unit 1)
-		(exclude_from_sim no)
-		(in_bom yes)
-		(on_board yes)
-		(dnp no)
-		(fields_autoplaced yes)
+		(at 104.14 41.91 0)
+		(mirror x)
+		(unit 1)
+		(exclude_from_sim no)
+		(in_bom yes)
+		(on_board yes)
+		(dnp no)
 		(property "Reference" "J3"
-			(at 105.41 39.3699 0)
+			(at 105.41 41.9101 0)
 			(effects
 				(font
@@
 		)
 		(property "Value" "Conn_01x02_Socket"
-			(at 105.41 41.9099 0)
-			(effects
-				(font
-					(size 1.27 1.27)
-				)
-				(justify left)
-			)
-		)
-		(property "Footprint" ""
-			(at 104.14 39.37 0)
+			(at 105.41 39.3701 0)
+			(effects
+				(font
+					(size 1.27 1.27)
+				)
+				(justify left)
+			)
+		)
+		(property "Footprint" "Connector_Molex:Molex_PicoBlade_53398-0271_1x02-1MP_P1.25mm_Vertical"
+			(at 104.14 41.91 0)
 			(effects
 				(font
@@
 		)
 		(property "Datasheet" "~"
-			(at 104.14 39.37 0)
+			(at 104.14 41.91 0)
 			(effects
 				(font
@@
 		)
 		(property "Description" "Generic connector, single row, 01x02, script generated"
-			(at 104.14 39.37 0)
-			(effects
-				(font
+			(at 104.14 41.91 0)
+			(effects
+				(font
+					(size 1.27 1.27)
+				)
+				(hide yes)
+			)
+		)
+		(property "LCSC" "C395343"
+			(at 104.14 41.91 0)
+			(effects
+				(font
