File: motor_unicorn.kicad_pcb (KiCad board)
At the start: 4 copper layers, 70 x 45 mm, 163 parts, among them J1 CON_SWD, J10 Conn_01x06_Pin, J11 Conn_01x02_Socket, J2 USB_C_Receptacle_USB2.0, J3 Conn_01x02_Socket, J4 Conn_01x02_Socket, J5 Conn_01x03_Socket, J6 Conn_01x03_Socket, J7 Conn_01x06_Pin, J8 Conn_01x06_Pin, J9 Conn_01x06_Pin, Q1 IPD068P03L3, Q10 Q_NMOS_SGD, Q11 Q_NMOS_SGD, Q12 Q_NMOS_SGD, Q13 Q_NMOS_SGD, Q2 Q_NMOS_SGD, Q3 Q_NMOS_SGD, Q4 Q_NMOS_SGD, Q5 Q_NMOS_SGD, Q6 Q_NMOS_SGD, Q7 Q_NMOS_SGD, Q8 Q_NMOS_SGD, Q9 Q_NMOS_SGD, U1 TLV62568DRL, U10 QMI8658, U11 EG2132, U12 EG2132, U13 EG2132, U14 INA240A1D, U15 INA240A1D, U16 OLED, U2 W25Q16JVUXIQ, U3 RP2040, U30 ADS1110, U31 LMR51420YDDCR, U4 EG2132, U5 EG2132, U6 EG2132, U7 INA240A1D, U8 INA240A1D, U9 SIT3088E, Y1 12MHz

Commit message: ordered version
Parts:
- added D22: D_Schottky, Diode_SMD:D_SOD-323, F.Cu at (-5.80, 6.70)
- C42, C47: footprint Capacitor_SMD:C_0402_1005Metric -> Capacitor_SMD:C_0805_2012Metric
- C45, C46: footprint Capacitor_SMD:C_0603_1608Metric -> Capacitor_SMD:C_0805_2012Metric
- U17: value ~ -> CJ9340
- Y1: footprint Crystal:Crystal_SMD_TXC_7M-4Pin_3.2x2.5mm -> Crystal:Crystal_SMD_3225-4Pin_3.2x2.5mm
- moved C42 2.41 mm to (8.20, -16.3)
- moved R1 1.90 mm to (-8.40, 7.40)
- moved R2 1.90 mm to (-8.40, 6.40)
- moved C25 1.87 mm to (-12.0, -0.10), turned to 0 degrees
- moved C45 1.71 mm to (5.50, 0.60)
- moved C47 1.32 mm to (-8.75, -3.60), turned to 0 degrees
- moved L1 0.61 mm to (-4.70, 9.20)
- moved C46 0.28 mm to (8.00, 8.20)
Connections:
- C49 pad 1: +5V -> Net-(D22-A)
- C50 pad 1: +5V -> Net-(D22-A)
- J2 pad A8: unconnected-(J2-SBU1-PadA8) -> (no net)
- J2 pad B8: unconnected-(J2-SBU2-PadB8) -> (no net)
- L3 pad 2: +5V -> Net-(D22-A)
- R31 pad 2: +5V -> Net-(D22-A)
Routing:
- net Net-(D22-A): track 0.00 -> 7.29 mm
- net +5V: track 51.1 -> 45.6 mm
- net GND: track 104.4 -> 101.6 mm
- net Net-(U16-VCOMH): track 3.25 -> 5.20 mm
- net /bridge/H_IN: track 17.3 -> 18.9 mm
- net /bridge/L_IN: track 16.9 -> 18.4 mm
- net VPP: track 5.76 -> 7.26 mm, vias 66 -> 65
- net +12V: track 100.2 -> 99.3 mm
- net Net-(U1-FB): track 2.37 -> 3.06 mm
- net +3V3: track 87.8 -> 87.5 mm, vias 25 -> 26

Commit message: tiny last minute fixes
Parts:
- added D23: 10V, Diode_SMD:D_SOD-323, F.Cu at (10.6, 8.20)
- added R35: 10k, Resistor_SMD:R_0402_1005Metric, F.Cu at (10.0, 9.70)
Connections:
- Q1 pad 1: GND -> Net-(D23-A)
Routing:
- net Net-(D23-A): track 0.00 -> 6.59 mm, vias 0 -> 1
- net VPP: track 7.26 -> 8.62 mm
- net GND: track 101.6 -> 100.3 mm
- net +12V: track 99.3 -> 98.7 mm
